File: smd-bb1to6.kicad_pcb (KiCad board)
At the start: 2 copper layers, 2 parts

Commit message: Initial version send to fabrication
Parts:
- removed the G*** at (22.4, 182.3)
- added ?: H1 2.54mm, Connector_PinHeader_2.54mm:PinHeader_1x06_P2.54mm_Vertical, F.Cu at (63.5, 124.5)
- added REF**: H2 2.54mm, Connector_PinHeader_2.54mm:PinHeader_1x06_P2.54mm_Vertical, F.Cu at (68.6, 124.5)
- added SOT-23-3: SOT-23, Package_TO_SOT_SMD:SOT-23, F.Cu at (76.5, 135.9)
- added SOT-23-6: SOT-23-6_Handsoldering, Package_TO_SOT_SMD:SOT-23-6_Handsoldering, F.Cu at (76.1, 125.4)
- moved G*** 72.9 mm to (78.7, 130.2)
Routing:
- net 3: track 0.00 -> 28.8 mm, vias 0 -> 1
- net 1: track 0.00 -> 26.7 mm, vias 0 -> 1
- net 2: track 0.00 -> 25.9 mm, vias 0 -> 1
- net 6: track 0.00 -> 25.4 mm
- net 5: track 0.00 -> 21.4 mm
- net 4: track 0.00 -> 16.3 mm
Other:
- board outline added: 20 x 20 mm
- board text added: "1"
- board text added: "2"
- board text added: "3"
- board text added: "4"
- board text added: "5"
- board text added: "6"
- board text added: "SOT23 3,5,6 BB v1.0 (2023)"
- board text added: "locked"
